File: throttle_encoder/throttle_encoder.kicad_sch (KiCad schematic)
At the start: 37 parts, among them J1 Conn_01x09_Shielded, P1 USB_C_Receptacle, P2 TC2030-CTX, SW1 INTERLOCK, SW2 SW_SPST, U1 STM32G0B1CBTx, U2 TCAN1044VDDFR, U3 AMS1117-3.3, Y1 ABM3-8MHZ, Y2 ABS07-32.768kHz

Commit message: Formatting
Parts:
- J1: value Conn_01x09_Shielded -> DSUB-9
Other:
- note added: "CAN"
- note added: "Input"
- note added: "MCU"
- note added: "Power"
- note added: "USB"
- moved on the sheet: C1, C10, C11, C12, C13, C14, C15, C16, C17, C2, C3, C4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

Commit message: Component selection
Parts:
- C13, C14, C15, C16, C17, C4, C5, C8: footprint (none) -> Capacitor_SMD:C_0603_1608Metric
- J1: footprint (none) -> Connector_Dsub:DSUB-9_Female_Vertical_P2.77x2.84mm_MountingHoles
- P2: footprint BlazeMicro:TC2030-IDC-NL -> Connector:Tag-Connect_TC2030-IDC-FP_2x03_P1.27mm_Vertical
- R4, R6, RV1: footprint (none) -> Resistor_SMD:R_0603_1608Metric
- SW1: footprint (none) -> Connector_Wago:Wago_734-132_1x02_P3.50mm_Vertical
- SW2: footprint (none) -> Button_Switch_SMD:SW_SPST_B3U-1000P
- Y1: footprint (none) -> Crystal:Crystal_SMD_Abracon_ABM3C-4Pin_5.0x3.2mm
- Y2: footprint (none) -> Crystal:Crystal_SMD_MicroCrystal_CC7V-T1A-2Pin_3.2x1.5mm
Changed lines of the file:
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@@
 	(label "CANTX"
 		(at 173.99 144.78 180)
+		(fields_autoplaced yes)
 		(effects
 			(font
@@
 	(label "CANRX"
 		(at 173.99 147.32 180)
+		(fields_autoplaced yes)
 		(effects
 			(font
@@
 	(label "CANH"
 		(at 247.65 146.05 180)
+		(fields_autoplaced yes)
 		(effects
 			(font
@@
 	(label "NRST"
 		(at 54.61 109.22 180)
+		(fields_autoplaced yes)
 		(effects
 			(font
@@
 	(label "CANTX"
 		(at 54.61 116.84 180)
+		(fields_autoplaced yes)
 		(effects
 			(font
@@
 	(label "CANL"
 		(at 265.43 129.54 180)
+		(fields_autoplaced yes)
 		(effects
 			(font
@@
 	(label "POT"
 		(at 160.02 100.33 0)
+		(fields_autoplaced yes)
 		(effects
 			(font
@@
 	(label "SWCLK"
 		(at 92.71 134.62 0)
+		(fields_autoplaced yes)
 		(effects
 			(font
@@
 	(label "D+"
 		(at 231.14 39.37 180)
+		(fields_autoplaced yes)
 		(effects
 			(font
@@
 	(label "INTERLOCK"
 		(at 92.71 101.6 0)
+		(fields_autoplaced yes)
 		(effects
 			(font
@@
 	(label "POT"
 		(at 92.71 99.06 0)
+		(fields_autoplaced yes)
 		(effects
 			(font
@@
 	(label "NRST"
 		(at 33.02 163.83 0)
+		(fields_autoplaced yes)
 		(effects
 			(font
@@
 	(label "CANRX"
 		(at 54.61 114.3 180)
+		(fields_autoplaced yes)
 		(effects
 			(font
@@
 	(label "D+"
 		(at 92.71 129.54 0)
+		(fields_autoplaced yes)
 		(effects
 			(font
@@
 	(label "SWCLK"
 		(at 95.25 76.2 0)
+		(fields_autoplaced yes)
 		(effects
 			(font
@@
 	(label "SWDIO"
 		(at 92.71 132.08 0)
+		(fields_autoplaced yes)
 		(effects
 			(font
@@
 	(label "D-"
 		(at 92.71 127 0)
+		(fields_autoplaced yes)
 		(effects
 			(font
@@
 	(label "CAN_STB"
 		(at 189.23 144.78 0)
+		(fields_autoplaced yes)
 		(effects
 			(font
@@
 	(label "CANL"
 		(at 247.65 135.89 180)
+		(fields_autoplaced yes)
 		(effects
 			(font
@@
 	(label "D-"
 		(at 231.14 36.83 180)
+		(fields_autoplaced yes)
 		(effects
 			(font
@@
 	(label "CANH"
 		(at 265.43 142.24 180)
+		(fields_autoplaced yes)
 		(effects
 			(font
@@
 	(label "SWDIO"
 		(at 95.25 73.66 0)
+		(fields_autoplaced yes)
 		(effects
 			(font
@@
 	(label "NRST"
 		(at 72.39 76.2 180)
+		(fields_autoplaced yes)
 		(effects
 			(font
@@
 	(label "INTERLOCK"
 		(at 180.34 100.33 180)
+		(fields_autoplaced yes)
 		(effects
 			(font
@@
 			)
 		)
-		(property "Footprint" ""
+		(property "Footprint" "Capacitor_SMD:C_0603_1608Metric"
 			(at 31.75 166.6748 0)
 			(effects
@@
 			)
 		)
-		(property "Footprint" ""
+		(property "Footprint" "Resistor_SMD:R_0603_1608Metric"
 			(at 156.21 100.33 0)
 			(effects
@@
 			)
 		)
-		(property "Footprint" ""
+		(property "Footprint" "Capacitor_SMD:C_0603_1608Metric"
 			(at 40.9448 43.18 0)
 			(effects
@@
 			)
 		)
-		(property "Footprint" ""
+		(property "Footprint" "Crystal:Crystal_SMD_Abracon_ABM3C-4Pin_5.0x3.2mm"
 			(at 27.94 105.41 0)
 			(effects
@@
 			)
 		)
-		(property "Footprint" ""
+		(property "Footprint" "Capacitor_SMD:C_0603_1608Metric"
 			(at 20.32 102.5652 0)
 			(effects
@@
 			)
 		)
-		(property "Footprint" ""
+		(property "Footprint" "Crystal:Crystal_SMD_MicroCrystal_CC7V-T1A-2Pin_3.2x1.5mm"
 			(at 26.67 135.89 0)
 			(effects
@@
 			)
 		)
-		(property "Footprint" ""
+		(property "Footprint" "Capacitor_SMD:C_0603_1608Metric"
 			(at 63.1952 43.18 0)
 			(effects
@@
 			)
 		)
-		(property "Footprint" ""
+		(property "Footprint" "Resistor_SMD:R_0603_1608Metric"
 			(at 182.626 96.774 90)
 			(effects
@@
 			)
 		)
-		(property "Footprint" ""
+		(property "Footprint" "Button_Switch_SMD:SW_SPST_B3U-1000P"
 			(at 27.94 163.83 0)
 			(effects
@@
 			)
 		)
-		(property "Footprint" ""
+		(property "Footprint" "Connector_Wago:Wago_734-132_1x02_P3.50mm_Vertical"
 			(at 194.31 100.33 0)
 			(effects
@@
 			)
 		)
-		(property "Footprint" ""
+		(property "Footprint" "Connector_Dsub:DSUB-9_Female_Vertical_P2.77x2.84mm_MountingHoles"
 			(at 270.51 137.16 0)
 			(effects
@@
 			)
 		)
-		(property "Footprint" ""
+		(property "Footprint" "Capacitor_SMD:C_0603_1608Metric"
 			(at 19.05 133.0452 0)
 			(effects
@@
 			)
 		)
-		(property "Footprint" ""
+		(property "Footprint" "Capacitor_SMD:C_0603_1608Metric"
 			(at 26.67 138.7348 0)
 			(effects
@@
 			)
 		)
-		(property "Footprint" ""
+		(property "Footprint" "Capacitor_SMD:C_0603_1608Metric"
 			(at 198.12 103.1748 0)
 			(effects
@@
 			)
 		)
-		(property "Footprint" "BlazeMicro:TC2030-IDC-NL"
+		(property "Footprint" "Connector:Tag-Connect_TC2030-IDC-FP_2x03_P1.27mm_Vertical"
 			(at 83.82 76.2 0)
 			(effects
@@
 			)
 		)
-		(property "Footprint" ""
+		(property "Footprint" "Capacitor_SMD:C_0603_1608Metric"
 			(at 27.94 108.2548 0)
 			(effects
@@
 			)
 		)
-		(property "Footprint" ""
+		(property "Footprint" "Resistor_SMD:R_0603_1608Metric"
 			(at 35.306 110.236 90)
 			(effects

Commit message: PCB Work
Parts:
- removed C10, C12: 0.1uF, Capacitor_SMD:C_0603_1608Metric, symbol Device:C
- removed C11: 1uF, Capacitor_SMD:C_0603_1608Metric, symbol Device:C
- removed C15, C16: 8pF, Capacitor_SMD:C_0603_1608Metric, symbol Device:C
- removed C9: 4.7uF, Capacitor_SMD:C_0603_1608Metric, symbol Device:C
- removed R4: 2.4k, Resistor_SMD:R_0603_1608Metric, symbol Device:R_US
- removed U1: STM32G0B1CBTx, Package_QFP:LQFP-48_7x7mm_P0.5mm, symbol MCU_ST_STM32G0:STM32G0B1CBTx
- removed U3: AMS1117-3.3, Package_TO_SOT_SMD:SOT-223-3_TabPin2, symbol Regulator_Linear:AMS1117-3.3
- removed Y1: ABM3-8MHZ, Crystal:Crystal_SMD_Abracon_ABM3C-4Pin_5.0x3.2mm, symbol Device:Crystal
- added C10, C9: 4.7nF, Capacitor_SMD:C_0402_1005Metric, symbol Device:C_Small
- added U3: STM32G0B1KBUx, Package_DFN_QFN:QFN-32-1EP_5x5mm_P0.5mm_EP3.45x3.45mm, symbol MCU_ST_STM32G0:STM32G0B1KBUx
- added U4: AP2112K-3.3, Package_TO_SOT_SMD:SOT-23-5, symbol Regulator_Linear:AP2112K-3.3
- C1, C13, C14, C17, C2, C3, C4, C5, C6, C7, C8: footprint Capacitor_SMD:C_0603_1608Metric -> Capacitor_SMD:C_0402_1005Metric
- R1, R2, R3, R6, R7, R8: footprint Resistor_SMD:R_0603_1608Metric -> Resistor_SMD:R_0402_1005Metric
- RV1: footprint Resistor_SMD:R_0603_1608Metric -> Potentiometer_THT:Potentiometer_Bourns_PTV09A-1_Single_Vertical
Connections:
- net +3V3: now also U3.4 (VDD), U4.5 (VOUT)
- net +5V: now also U4.1 (VIN), U4.3 (EN)
- net CANH: now also D1.2 (K2), C10.1; no longer D1.1 (K1)
- net CANL: now also D1.1 (K1), C9.1; no longer D1.2 (K2)
- net CANRX: now also U3.29 (PB5)
- net CANTX: now also U3.30 (PB6)
- net D+: now also U3.23 (PA12/PA10)
- net D-: now also U3.22 (PA11/PA9)
- net GND: now also C10.2, C9.2, U3.33 (VSS), U3.5 (VSS), U4.2 (GND)
- net INTERLOCK: now also U3.8 (PA1)
- net NRST: now also U3.6 (PF2)
- net POT: now also U3.7 (PA0)
- net SWCLK: now also U3.25 (PA14)
- net SWDIO: now also U3.24 (PA13)
- net at C14.2, Y2.1: now also U3.3 (PC15)
- net at C13.1, Y2.2: now also U3.2 (PC14)
- no-connect marks 39 -> 8
Other:
- moved on the sheet: C13, C14, C4, C5, Y2

Commit message: Finishing touches
Parts:
- removed FL1: Choke, Inductor_SMD:L_CommonModeChoke_Coilcraft_0603USB, symbol Filter:Choke_Coilcraft_0603USB-142
- removed SW1: INTERLOCK, Connector_Wago:Wago_734-132_1x02_P3.50mm_Vertical, symbol Switch:SW_SPST
- added FL1: Choke, railspeeder:DLW32PH_MUR, symbol Railspeeder:DLW32SH510XF2L
- added J2: 2601-1102, railspeeder:CONN2_2601-1102_WAG, symbol Railspeeder:2601-1102
- renumbered C5 to C1, C17 to C11, C1 to C12, C2 to C13, C4 to C2, C14 to C3, C9 to C4, C13 to C5, C3 to C7, C7 to C9, P2 to P1, P1 to P2, R3 to R2, R6 to R3, R7 to R4, R8 to R5, R2 to R6, SW2 to SW1, U4 to U1, U3 to U2, U2 to U3, Y2 to Y1
Connections:
- net CANH: now also FL1.2
- net CANL: now also FL1.3
- net GND: now also J2.1 (1_1), J2.2 (1_2)
- net INTERLOCK: now also J2.3 (2_1), J2.4 (2_2)
- net at U3.6 (CANL): now also FL1.4
- net at U3.7 (CANH): now also FL1.1
Other:
- moved on the sheet: C13, C7, R2, U3

Commit message: Finishing touches
Parts:
- renumbered C9 to C10, C10 to C11, C11 to C12, C12 to C13, C13 to C9
Changed lines of the file:
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@@
 		(on_board yes)
 		(dnp no)
-		(property "Reference" "C10"
+		(property "Reference" "C11"
 			(at 221.488 147.32 90)
 			(effects
@@
 			(project "throttle_encoder"
 				(path "/e24a3f1a-dec4-4fc0-b25c-13b39bb3b7cd"
-					(reference "C10")
+					(reference "C11")
 					(unit 1)
 				)
@@
 		(on_board yes)
 		(dnp no)
-		(property "Reference" "C13"
+		(property "Reference" "C9"
 			(at 138.43 140.9699 0)
 			(effects
@@
 			(project "throttle_transcoder"
 				(path "/e24a3f1a-dec4-4fc0-b25c-13b39bb3b7cd"
-					(reference "C13")
+					(reference "C9")
 					(unit 1)
 				)
@@
 		(on_board yes)
 		(dnp no)
-		(property "Reference" "C12"
+		(property "Reference" "C13"
 			(at 222.25 138.684 90)
 			(effects
@@
 			(project "throttle_transcoder"
 				(path "/e24a3f1a-dec4-4fc0-b25c-13b39bb3b7cd"
-					(reference "C12")
+					(reference "C13")
 					(unit 1)
 				)
@@
 		(dnp no)
 		(fields_autoplaced yes)
-		(property "Reference" "C9"
+		(property "Reference" "C10"
 			(at 91.44 38.0999 0)
 			(effects
@@
 			(project "throttle_transcoder"
 				(path "/e24a3f1a-dec4-4fc0-b25c-13b39bb3b7cd"
-					(reference "C9")
+					(reference "C10")
 					(unit 1)
 				)
@@
 		(on_board yes)
 		(dnp no)
-		(property "Reference" "C11"
+		(property "Reference" "C12"
 			(at 188.468 103.378 90)
 			(effects
@@
 			(project "throttle_transcoder"
 				(path "/e24a3f1a-dec4-4fc0-b25c-13b39bb3b7cd"
-					(reference "C11")
-					(unit 1)
-				)
+					(reference "C12")
+					(unit 1)
+				)
