File: can-backplane/can-backplane.kicad_pcb (KiCad board)
At the start: 4 copper layers, 70 x 240 mm, 58 parts, among them J1 BATT, J10 DSUB-9, J11 DSUB-9, J12 Raspberry_Pi, J13 DSUB-9, J14 DSUB-9, J15 DSUB-9, J16 DSUB-9, J17 DSUB-9, J18 DSUB-9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

Commit message: PCB Work
Parts:
- added C21: 4.7nF, Capacitor_SMD:C_0603_1608Metric, F.Cu at (67.4, 70.7)
- added C22: 4.7nF, Capacitor_SMD:C_0603_1608Metric, F.Cu at (67.4, 74.7)
- added R7: 5.1k, Resistor_SMD:R_0603_1608Metric, F.Cu at (60.0, 70.7)
- J1: footprint Connector_PinSocket_2.54mm:PinSocket_1x02_P2.54mm_Vertical -> TerminalBlock_WAGO:TerminalBlock_WAGO_236-102_1x02_P5.00mm_45Degree
- moved J22 489.7 mm to (253.2, 98.4), turned to 90 degrees
- moved J21 473.5 mm to (237.7, 98.4), turned to 90 degrees
- moved J11 459.4 mm to (253.2, 64.6), turned to 90 degrees
- moved J20 457.9 mm to (222.2, 98.4), turned to 90 degrees
- moved J19 442.7 mm to (206.7, 98.4), turned to 90 degrees
- moved J10 442.1 mm to (237.7, 64.6), turned to 90 degrees
- moved J18 428.4 mm to (191.2, 98.6), turned to 90 degrees
- moved J9 425.5 mm to (222.2, 64.9), turned to 90 degrees
- moved J17 414.5 mm to (175.7, 98.6), turned to 90 degrees
- moved J8 409.2 mm to (206.7, 64.9), turned to 90 degrees
- moved C14 406.5 mm to (52.6, 75.0), turned to 180 degrees
- moved C15 403.1 mm to (52.6, 69.5), turned to 180 degrees
- moved C1 402.8 mm to (67.4, 72.7)
- moved U3 402.7 mm to (46.6, 72.7), turned to 180 degrees
- moved J16 401.3 mm to (160.2, 98.6), turned to 90 degrees
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Connections:
- C17 pad 1: +3V3 -> Net-(U4-V+)
- C17 pad 2: Net-(U4-V+) -> GND
Routing:
- net Net-(U4-C1-): track 0.00 -> 3.93 mm
- net Net-(U4-C1+): track 0.00 -> 3.69 mm
- net Net-(U4-V+): track 0.00 -> 2.32 mm
- net Net-(U4-V-): track 0.00 -> 2.26 mm
- net Net-(U4-C2-): track 0.00 -> 2.18 mm
- net Net-(U4-C2+): track 0.00 -> 2.06 mm
Other:
- board size 70 x 240 mm -> 240 x 70 mm

Commit message: PCB Work
Parts:
- moved C16 6.33 mm to (82.3, 82.5)
- moved C17 6.33 mm to (90.1, 82.5)
- moved C18 6.33 mm to (89.1, 81.0)
- moved C19 6.33 mm to (85.3, 82.5)
- moved C20 6.33 mm to (89.3, 91.5)
- moved U4 6.33 mm to (85.5, 87.0)
- moved R5 5.91 mm to (88.7, 75.8), turned to 0 degrees
- moved R3 3.64 mm to (85.4, 75.8), turned to 0 degrees
- moved C10 2.81 mm to (80.5, 73.0)
- moved C11 2.81 mm to (79.0, 73.0)
- moved C12 2.81 mm to (77.5, 73.0)
- moved C8 2.81 mm to (83.5, 73.0)
- moved C9 2.81 mm to (82.0, 73.0)
- moved D2 2.81 mm to (79.0, 70.0)
- moved L1 2.81 mm to (84.0, 69.0)
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Connections:
- C10 pad 2: Net-(D2-K) -> GND
- C11 pad 2: Net-(D2-K) -> GND
- C12 pad 2: Net-(D2-K) -> GND
- C5 pad 2: Net-(D2-K) -> GND
- C6 pad 2: Net-(D2-K) -> GND
- C7 pad 2: Net-(D2-K) -> GND
- C8 pad 2: Net-(D2-K) -> GND
- C9 pad 2: Net-(D2-K) -> GND
- D1 pad 1: /CANH -> /CANL
- D1 pad 2: /CANL -> /CANH
- D2 pad 1: Net-(D2-K) -> GND
- J1 pad 2: Net-(D2-K) -> GND
- J12 pad 18: /INT0 -> /INT1
- J12 pad 22: /INT1 -> /INT0
- R5 pad 2: Net-(D2-K) -> GND
- U1 pad 3: Net-(D2-K) -> GND
- U1 pad 4: Net-(D2-K) -> GND
Routing:
- net /CANH: track 0.00 -> 375.2 mm, vias 0 -> 1
- net /CANL: track 0.00 -> 370.2 mm, vias 0 -> 1
- net +3V3: track 0.00 -> 89.2 mm, vias 0 -> 4
- net /RX: track 0.00 -> 38.8 mm
- net /TX: track 0.00 -> 36.2 mm
- net GND: track 0.00 -> 25.3 mm, vias 0 -> 29
- net /INT: track 0.00 -> 23.6 mm, vias 0 -> 1
- net /INT1: track 0.00 -> 23.3 mm
- net VBUS: track 0.00 -> 21.5 mm
- net /INT0: track 0.00 -> 20.4 mm
- net /CS: track 0.00 -> 19.9 mm, vias 0 -> 1
- net /SCK: track 0.00 -> 18.0 mm, vias 0 -> 1
- net /MOSI: track 0.00 -> 15.8 mm, vias 0 -> 1
- net Net-(J23-Pin_2): track 0.00 -> 14.5 mm
- net Net-(J23-Pin_3): track 0.00 -> 12.5 mm
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- added copper zone on F.Cu, net +5V
- added copper zone on F.Cu, net GND
- added copper zone on F.Cu, net Net-(U1-SW)
- added copper zone on F.Cu, net VBUS

Commit message: PCB Work
Parts:
- J12: moved to F.Cu
- turned J12 to 0 degrees
Routing:
- net /MOSI: track 15.8 -> 46.2 mm
- net /MISO: track 12.2 -> 42.3 mm
- net /SCK: track 18.0 -> 46.9 mm
- net /RX: track 38.8 -> 67.3 mm, vias 0 -> 1
- net /TX: track 36.2 -> 63.1 mm, vias 0 -> 1
- net +3V3: track 89.2 -> 69.4 mm
- net /CS: track 19.9 -> 30.6 mm
- net /INT: track 23.6 -> 13.8 mm, vias 1 -> 2
- net /INT0: track 20.4 -> 26.6 mm, vias 0 -> 1
- net /CAN_STB: track 10.0 -> 10.6 mm
- net /INT1: track 23.3 -> 23.6 mm, vias 0 -> 1
